Commit message: Robot Actualizado

File: src/robot_ERA/urdf/robot_ERA.urdf (robot description, URDF)
Before this commit: robot robot_ERA, 8 links, 7 joints
Links:
- link link_0: geometry collision mesh filename=package://Robot_ERA/meshes/link_0.STL; visual mesh filename=package://Robot_ERA/meshes/link_0.STL
- link link_1: geometry collision mesh filename=package://Robot_ERA/meshes/link_1.STL; visual mesh filename=package://Robot_ERA/meshes/link_1.STL
- link link_2: mass 2.9774 -> 2.97737093271591; geometry collision mesh filename=package://Robot_ERA/meshes/link_2.STL; visual mesh filename=package://Robot_ERA/meshes/link_2.STL
- link link_3: mass 1.4008 -> 1.40082730035319; geometry collision mesh filename=package://Robot_ERA/meshes/link_3.STL; visual mesh filename=package://Robot_ERA/meshes/link_3.STL
- link link_4: mass 0.34675 -> 0.346752223723456; geometry collision mesh filename=package://Robot_ERA/meshes/link_4.STL; visual mesh filename=package://Robot_ERA/meshes/link_4.STL
- link link_5: mass 0.15564 -> 0.155635640889723; geometry collision mesh filename=package://Robot_ERA/meshes/link_5.STL; visual mesh filename=package://Robot_ERA/meshes/link_5.STL
- link link_6_1: mass 0.019387 -> 0.01938707412012; geometry collision mesh filename=package://Robot_ERA/meshes/link_6_1.STL; visual mesh filename=package://Robot_ERA/meshes/link_6_1.STL
- link link_6_2: mass 0.019424 -> 0.0194236693750671; geometry collision mesh filename=package://Robot_ERA/meshes/link_6_2.STL; visual mesh filename=package://Robot_ERA/meshes/link_6_2.STL
Joints:
- joint joint_1: limit lower=-1.5708 upper=1.5708 effort=1000 velocity=5 -> lower=-2.3562 upper=2.3562 effort=1000 velocity=5
- joint joint_2: limit lower=-1.5708 upper=1.5708 effort=1000 velocity=5 -> lower=-1.5708 upper=1.5708 effort=45.1 velocity=0.114
- joint joint_3: limit lower=-1.5708 upper=1.5708 effort=1000 velocity=5 -> lower=-3.927 upper=0.7854 effort=22.7 velocity=0.114
- joint joint_4: limit lower=-1.5708 upper=1.5708 effort=1000 velocity=5 -> lower=-2.3562 upper=2.3562 effort=0.5 velocity=8
- joint joint_5: limit lower=-1.5708 upper=1.5708 effort=1000 velocity=5 -> lower=-3.927 upper=0.7854 effort=0.35 velocity=2
- joint joint_6_1: limit lower=0 upper=0.1 effort=100 velocity=5 -> lower=0 upper=0.05 effort=0.1 velocity=0.05
- joint joint_6_2: limit lower=0 upper=0.1 effort=100 velocity=5 -> lower=0 upper=0.05 effort=0.1 velocity=0.05
