Commit message: Se añadieron correctamente los límites del robot ERA en base a los motores originales

File: src/ERA/urdf/ERA.urdf (robot description, URDF)
Before this commit: robot Robot_ERA, 8 links, 7 joints
Links:
- link link_0: geometry collision mesh filename=package://ERA/meshes/link_0.STL; visual mesh filename=package://ERA/meshes/link_0.STL
- link link_1: geometry collision mesh filename=package://ERA/meshes/link_1.STL; visual mesh filename=package://ERA/meshes/link_1.STL
- link link_2: mass 2.97737093271591 -> 2.9773709327159; geometry collision mesh filename=package://ERA/meshes/link_2.STL; visual mesh filename=package://ERA/meshes/link_2.STL
- link link_3: geometry collision mesh filename=package://ERA/meshes/link_3.STL; visual mesh filename=package://ERA/meshes/link_3.STL
- link link_4: geometry collision mesh filename=package://ERA/meshes/link_4.STL; visual mesh filename=package://ERA/meshes/link_4.STL
- link link_5: mass 0.155635640889723 -> 0.15564; geometry collision mesh filename=package://ERA/meshes/link_5.STL; visual mesh filename=package://ERA/meshes/link_5.STL
- link link_6_1: mass 0.01938707412012 -> 0.019387; geometry collision mesh filename=package://ERA/meshes/link_6_1.STL; visual mesh filename=package://ERA/meshes/link_6_1.STL
- link link_6_2: mass 0.0194236693750671 -> 0.019424; geometry collision mesh filename=package://ERA/meshes/link_6_2.STL; visual mesh filename=package://ERA/meshes/link_6_2.STL
Joints:
- joint joint_1: limit lower=-2.3562 upper=2.3562 effort=1000 velocity=5 -> lower=-2.3562 upper=2.3562 effort=7.1537 velocity=0.2188; origin xyz=0 0 0.18918 rpy=-1.5708 0 -1.5708 -> xyz=0 0 0.189175 rpy=-1.5707963267949 0 -1.57079632679489
- joint joint_2: limit lower=-1.5708 upper=1.5708 effort=45.1 velocity=0.114 -> lower=-1.5708 upper=1.5708 effort=86.211 velocity=0.1163; origin xyz=0.00012374 -0.25568 0.00149 rpy=0 0 -1.5708 -> xyz=0.000123744699244387 -0.25567672725 0.00148999999984069 rpy=0 0 -1.5707963267949
- joint joint_3: limit lower=-3.927 upper=0.7854 effort=22.7 velocity=0.114 -> lower=-3.927 upper=0.7854 effort=24.654 velocity=0.0635; origin xyz=0 0 0 rpy=-1.5708 0 0 -> xyz=0 0 0 rpy=-1.5707963267949 0 0
- joint joint_4: limit lower=-2.3562 upper=2.3562 effort=0.5 velocity=8 -> lower=-2.3562 upper=2.3562 effort=15.93 velocity=0.0982; origin xyz=0 0 0.4284 rpy=-1.5708 0 -3.1416 -> xyz=0 0 0.428399999999979 rpy=-1.57079632679491 0 -3.1415926535893
- joint joint_5: limit lower=-3.927 upper=0.7854 effort=0.35 velocity=2 -> lower=-3.927 upper=0.7854 effort=3.5 velocity=7.48
- joint joint_6_1: limit lower=0 upper=0.05 effort=0.1 velocity=0.05 -> lower=0 upper=0.32 effort=218.75 velocity=0.016
- joint joint_6_2: limit lower=0 upper=0.05 effort=0.1 velocity=0.05 -> lower=0 upper=0.05 effort=218.75 velocity=0.016
