Commit message: modificacion archivo proyecto final

File: src/robotchino/urdf/robotchino.urdf (robot description, URDF)
Before this commit: robot robotchino, 9 links, 8 joints
Links:
- link magnet_link: mass 3 -> 3.0

Commit message: se añadio el codigo de la tortuga

File: src/robotchino/urdf/robotchino.urdf (robot description, URDF)
Before this commit: robot robotchino, 9 links, 8 joints
Links:
- removed link magnet_link
Joints:
- removed joint magnet_joint
